File: SAI/board.kicad_pcb (KiCad board)
At the start: 2 copper layers, 122.3 x 101.1 mm, 47 parts, among them J1 Jumper, J2 Jumper

Commit message: Code cleanup
Parts:
- removed B1: , kbd:ResetSW
- removed J1, J2: Jumper, lib:Jumper
- removed MCU1, MCU2: , ProMicro
- removed PAD1, PAD2: , SMDPad
- removed T1, T2: , E73:SPDT_C128955
