File: SAI/board.kicad_pcb (KiCad board)
At the start: 2 copper layers, 122.3 x 101.1 mm, 38 parts

Commit message: Working PCB with 6 DRC warnings
Parts:
- removed TRRS1, TRRS2: TRRS-PJ-320A-dual, TRRS-PJ-320A-dual
- added D19: , ComboDiode, F.Cu at (261.4, 5.00)
- added D20: , ComboDiode, F.Cu at (261.4, -14.1)
- added D21: , ComboDiode, F.Cu at (261.4, -33.1)
- added D22: , ComboDiode, F.Cu at (242.4, -8.34)
- added D23: , ComboDiode, F.Cu at (242.4, -27.4)
- added D24: , ComboDiode, F.Cu at (242.4, -46.4)
- added D25: , ComboDiode, F.Cu at (223.3, -12.1)
- added D26: , ComboDiode, F.Cu at (223.3, -31.2)
- added D27: , ComboDiode, F.Cu at (223.3, -50.2)
- added D28: , ComboDiode, F.Cu at (204.3, -8.34)
- added D29: , ComboDiode, F.Cu at (204.3, -27.4)
- added D30: , ComboDiode, F.Cu at (204.3, -46.4)
- added D31: , ComboDiode, F.Cu at (185.2, -6.43)
- added D32: , ComboDiode, F.Cu at (185.2, -25.5)
- added D33: , ComboDiode, F.Cu at (185.2, -44.5)
- added D34: , ComboDiode, F.Cu at (194.3, 17.7)
- added D35: , ComboDiode, F.Cu at (175.7, 25.4)
- added D36: , ComboDiode, F.Cu at (159.8, 37.6)
- added MCU1: RPi_Pico_SMD_TH, MCU_RaspberryPi_and_Boards:RPi_Pico_SMD_TH, F.Cu at (139.2, -32.5)
- added S19: , MX, F.Cu at (261.4, 0.00)
- added S20: , MX, F.Cu at (261.4, -19.1)
- added S21: , MX, F.Cu at (261.4, -38.1)
- added S22: , MX, F.Cu at (242.4, -13.3)
- added S23: , MX, F.Cu at (242.4, -32.4)
- added S24: , MX, F.Cu at (242.4, -51.4)
- added S25: , MX, F.Cu at (223.3, -17.1)
- added S26: , MX, F.Cu at (223.3, -36.2)
- added S27: , MX, F.Cu at (223.3, -55.2)
- added S28: , MX, F.Cu at (204.3, -13.3)
- added S29: , MX, F.Cu at (204.3, -32.4)
- added S30: , MX, F.Cu at (204.3, -51.4)
- added S31: , MX, F.Cu at (185.2, -11.4)
- added S32: , MX, F.Cu at (185.2, -30.5)
- added S33: , MX, F.Cu at (185.2, -49.5)
- added S34: , MX, F.Cu at (193.0, 12.9)
- added S35: , MX, F.Cu at (173.2, 21.1)
- added S36: , MX, F.Cu at (156.3, 34.1)
- S1, S10, S11, S12, S13, S14, S15, S16, S17, S18, S2, S3, S4, S5, S6, S7, S8, S9: footprint PG1350 -> MX
- moved D18 8.37 mm to (120.7, 37.6)
- moved S18 8.37 mm to (124.2, 34.1)
- moved D15 7.48 mm to (95.2, -44.5)
- moved S15 7.48 mm to (95.2, -49.5)
- moved S17 7.07 mm to (107.3, 21.1)
- moved D17 7.07 mm to (104.8, 25.4)
- moved D12 6.95 mm to (76.2, -46.4)
- moved S12 6.95 mm to (76.2, -51.4)
- moved D9 6.73 mm to (57.1, -50.2)
- moved S9 6.73 mm to (57.1, -55.2)
- moved D14 6.19 mm to (95.2, -25.5)
- moved S14 6.19 mm to (95.2, -30.5)
- moved D6 5.92 mm to (38.1, -46.4)
- moved S6 5.92 mm to (38.1, -51.4)
- moved S16 5.79 mm to (87.5, 12.9)
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Connections:
- net P14 renamed C5
- net P15 renamed C4
- net P18 renamed C3
- net P19 renamed C2
- net P20 renamed C1
- D1 pad 1: pinky_bottom -> R3
- D1 pad 2: P6 -> R3
- D10 pad 2: P6 -> R3
- D11 pad 1: index_home -> R2
- D11 pad 2: P5 -> index_home
- D12 pad 1: index_top -> R1
- D12 pad 2: P4 -> R1
- D13 pad 1: inner_bottom -> R3
- D13 pad 2: P6 -> inner_bottom
- D14 pad 1: inner_home -> R2
- D14 pad 2: P5 -> inner_home
- D15 pad 2: P4 -> inner_top
- D16 pad 2: P7 -> R4
- D17 pad 2: P7 -> home_thumb
- D18 pad 1: far_thumb -> R4
- D18 pad 2: P7 -> far_thumb
- D2 pad 2: P5 -> R2
- D3 pad 2: P4 -> pinky_top
- D4 pad 1: ring_bottom -> R3
- D4 pad 2: P6 -> R3
- D5 pad 2: P5 -> ring_home
- D6 pad 1: ring_top -> R1
- D6 pad 2: P4 -> ring_top
- D7 pad 1: middle_bottom -> R3
- D7 pad 2: P6 -> R3
- D8 pad 2: P5 -> R2
- D9 pad 2: P4 -> R1
Routing:
- net R3: track 0.00 -> 338.5 mm, vias 0 -> 1
- net R2: track 0.00 -> 296.1 mm
- net R1: track 0.00 -> 290.5 mm
- net C7: track 0.00 -> 201.1 mm, vias 0 -> 2
- net C8: track 0.00 -> 199.1 mm, vias 0 -> 3
- net C9: track 0.00 -> 198.4 mm, vias 0 -> 1
- net C10: track 0.00 -> 195.6 mm, vias 0 -> 1
- net C1: track 0.00 -> 187.4 mm, vias 0 -> 2
- net R4: track 0.00 -> 187.0 mm
- net C6: track 0.00 -> 184.9 mm, vias 0 -> 2
- net C3: track 0.00 -> 181.9 mm
- net C5: track 0.00 -> 170.9 mm, vias 0 -> 1
- net C4: track 0.00 -> 156.0 mm, vias 0 -> 2
- net C2: track 0.00 -> 145.7 mm, vias 0 -> 1
- net inner_bottom: track 0.00 -> 22.3 mm, vias 0 -> 1
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Other:
- board size 122.3 x 101.1 mm -> 263.5 x 114.3 mm
- net class Default removed
- net class Power removed
- board text added: "BRAILLE Keyboard v0.1"
- board text removed: "BRAILLE Keyboard v0.1 by shaggyshelar"
